Commit message: added vision

File: human_robot_collision_RL/data/walls.urdf (robot description, URDF)
Before this commit: robot walls, 3 links, 2 joints
Links:
- link left_wall: geometry collision box size=0.1 30.0 2.0; visual box size=0.1 30.0 2.0
- link right_wall: geometry collision box size=0.1 30.0 2.0; visual box size=0.1 30.0 2.0
Joints:
- joint back_to_left_wall: origin xyz=-0.95 4.95 0.0 -> xyz=-0.95 14.95 0.0
- joint back_to_right_wall: origin xyz=0.95 4.95 0.0 -> xyz=0.95 14.95 0.0
